File: IM6100 HID.kicad_pcb (KiCad board)
At the start: 2 copper layers, 100 x 80 mm, 79 parts, among them J3 Expansion Header, SW1 DX0, SW10 DX9, SW11 DX10, SW12 DX11, SW2 DX1, SW3 DX2, SW4 DX3, SW5 DX4, SW6 DX5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

Commit message: HID board finalizing
Parts:
- removed U11, U12, U13: 74LS125, Package_SO:SO-14_3.9x8.65mm_P1.27mm
- added C6: 100n, Capacitor_SMD:C_0805_2012Metric_Pad1.18x1.45mm_HandSolder, F.Cu at (194.3, 109.2)
- added C7: 100n, Capacitor_SMD:C_0805_2012Metric_Pad1.18x1.45mm_HandSolder, F.Cu at (160.0, 116.8)
- added R37: 10k, Resistor_SMD:R_0805_2012Metric, F.Cu at (192.3, 148.6)
- added R38: 100k, Resistor_SMD:R_0805_2012Metric, F.Cu at (194.3, 114.3)
- added SW13: STEP MODE, Connector_PinHeader_2.54mm:PinHeader_1x03_P2.54mm_Vertical, F.Cu at (186.7, 148.6)
- added SW14: INSTR STEP, Button_Switch_THT:SW_PUSH_6mm_H4.3mm, F.Cu at (190.4, 127.0)
- added U14: 74HC74, Package_SO:SO-14_3.9x8.65mm_P1.27mm, F.Cu at (191.1, 138.5)
- added U15: 74HC541, Package_SO:SO-20_12.8x7.5mm_P1.27mm, F.Cu at (128.8, 139.0)
- added U16: 74HC541, Package_SO:SO-20_12.8x7.5mm_P1.27mm, F.Cu at (162.7, 139.0)
- C1, C2, C3, C4, C5: footprint Capacitor_THT:C_Disc_D3.8mm_W2.6mm_P2.50mm -> Capacitor_SMD:C_0805_2012Metric_Pad1.18x1.45mm_HandSolder
- J3: value Expansion Header -> Expansion port; footprint Connector_IDC:IDC-Header_2x15_P2.54mm_Vertical -> Connector_PinHeader_2.54mm:PinHeader_2x16_P2.54mm_Vertical
- moved C3 87.2 mm to (119.6, 135.1), turned to -90 degrees
- moved C1 83.4 mm to (121.9, 104.6), turned to 180 degrees
- moved C4 52.5 mm to (153.4, 135.1), turned to -90 degrees
- moved C2 21.7 mm to (183.6, 116.8)
- moved C5 16.8 mm to (188.5, 132.3)
- moved U10 12.7 mm to (179.1, 138.5)
- moved SW1 7.62 mm to (114.3, 148.6)
- moved SW11 7.62 mm to (171.4, 148.6)
- moved SW12 7.62 mm to (177.2, 148.6)
- moved SW2 7.62 mm to (120.0, 148.6)
- moved SW4 7.62 mm to (131.4, 148.6)
- moved SW5 7.62 mm to (137.2, 148.6)
- moved SW6 7.62 mm to (142.9, 148.6)
- moved SW7 7.62 mm to (148.6, 148.6)
- moved SW8 7.62 mm to (154.3, 148.6)
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- renumbered HOLE3 to HOLE1, HOLE3 to HOLE2, HOLE3 to HOLE4
Connections:
- J3 pad 10: DX10 -> /C0
- J3 pad 11: DX9 -> DX11
- J3 pad 12: DX8 -> DX10
- J3 pad 13: DX7 -> DX9
- J3 pad 14: DX6 -> DX8
- J3 pad 15: /DEVSEL -> DX7
- J3 pad 16: /SWSEL -> DX6
- J3 pad 17: XTA -> /DEVSEL
- J3 pad 18: LXMAR -> /SWSEL
- J3 pad 19: XTB -> XTA
- J3 pad 20: XTC -> LXMAR
- J3 pad 21: READ2 -> XTB
- J3 pad 22: WRITE2 -> XTC
- J3 pad 23: DX5 -> READ2
- J3 pad 24: DX4 -> WRITE2
- J3 pad 25: DX3 -> DX5
- J3 pad 26: DX2 -> DX4
- J3 pad 27: DX1 -> DX3
- J3 pad 28: DX0 -> DX2
- J3 pad 29: TXD -> DX1
- J3 pad 30: SENSE3/RXD -> DX0
- J3 pad 5: /SKP -> /WAIT
- J3 pad 6: /C2 -> /RESET
- J3 pad 7: /C1 -> /SKP
- J3 pad 8: /C0 -> /C2
- J3 pad 9: DX11 -> /C1
- U10 pad 10: (no net) -> Net-(U10-Pad10)
- U10 pad 11: (no net) -> unconnected-(U10-Pad11)
- U10 pad 12: (no net) -> GND
- U10 pad 13: (no net) -> GND
- U10 pad 4: (no net) -> IFETCH
- U10 pad 5: (no net) -> Net-(C6-Pad1)
- U10 pad 6: (no net) -> Net-(U10-Pad10)
- U10 pad 8: (no net) -> Net-(U14A-C)
- U10 pad 9: (no net) -> Net-(U10-Pad10)
Routing:
- net /RESET: track 0.00 -> 131.2 mm, vias 0 -> 2
- net XTB: track 0.00 -> 127.2 mm, vias 0 -> 1
- net /WAIT: track 0.00 -> 124.2 mm
- net DX11: track 0.00 -> 105.6 mm, vias 0 -> 4
- net IFETCH: track 0.00 -> 105.6 mm, vias 0 -> 2
- net LXMAR: track 0.00 -> 99.0 mm, vias 0 -> 4
- net DX9: track 0.00 -> 97.1 mm, vias 0 -> 4
- net /SWSEL: track 0.00 -> 97.1 mm, vias 0 -> 4
- net DX10: track 0.00 -> 93.4 mm, vias 0 -> 4
- net DX8: track 0.00 -> 89.4 mm, vias 0 -> 4
- net DX7: track 0.00 -> 84.5 mm, vias 0 -> 4
- net DX5: track 0.00 -> 83.0 mm, vias 0 -> 4
- net DX6: track 0.00 -> 82.0 mm, vias 0 -> 4
- net /EL: track 0.00 -> 76.6 mm, vias 0 -> 2
- net DX3: track 0.00 -> 75.8 mm, vias 0 -> 4
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- added copper zone on F.Cu, net +5V
- added copper zone on B.Cu, net GND
Other:
- board text added: "0"
- board text added: "1"
- board text added: "DX0..2"
- board text added: "DX3..5"
- board text added: "DX6..8"
- board text added: "DX9..11"
- board text added: "IM6100 HID board"
- board text added: "OFF"
- board text added: "ON"
