File: IM6100 HID.kicad_sch (KiCad schematic)
At the start: 1 part, among them J3 Expansion Header

Commit message: HID board finalizing
Parts:
- removed J3: Expansion Header, Connector_IDC:IDC-Header_2x15_P2.54mm_Vertical, symbol Connector_Generic:Conn_02x15_Odd_Even
- added J3: Expansion port, Connector_PinHeader_2.54mm:PinHeader_2x16_P2.54mm_Vertical, symbol Connector_Generic:Conn_02x16_Odd_Even
Connections:
- net +5V: now also J3.1 (Pin_1)
- net /C0: now also J3.10 (Pin_10)
- net /C1: now also J3.9 (Pin_9)
- net /C2: now also J3.8 (Pin_8)
- net /DEVSEL: now also J3.17 (Pin_17)
- net /MEMSEL: now also J3.3 (Pin_3)
- net /SKP: now also J3.7 (Pin_7)
- net /SWSEL: now also J3.18 (Pin_18)
- net DX0: now also J3.30 (Pin_30)
- net DX1: now also J3.29 (Pin_29)
- net DX10: now also J3.12 (Pin_12)
- net DX11: now also J3.11 (Pin_11)
- net DX2: now also J3.28 (Pin_28)
- net DX3: now also J3.27 (Pin_27)
- net DX4: now also J3.26 (Pin_26)
- net DX5: now also J3.25 (Pin_25)
- net DX6: now also J3.16 (Pin_16)
- net DX7: now also J3.15 (Pin_15)
- net DX8: now also J3.14 (Pin_14)
- net DX9: now also J3.13 (Pin_13)
- net GND: now also J3.2 (Pin_2)
- net IFETCH: now also J3.4 (Pin_4)
- net LXMAR: now also J3.20 (Pin_20)
- net READ2: now also J3.23 (Pin_23)
- net SENSE3/RXD: now also J3.32 (Pin_32)
- net TXD: now also J3.31 (Pin_31)
- net WRITE2: now also J3.24 (Pin_24)
- net XTA: now also J3.19 (Pin_19)
- net XTB: now also J3.21 (Pin_21)
- net XTC: now also J3.22 (Pin_22)
- new net /RESET: J3.6 (Pin_6)
- new net /WAIT: J3.5 (Pin_5)
Other:
- added sheet Single instruction mode (HID single instruction.kicad_sch)
