File: IM6100 SAMPLER_v3.kicad_pcb (KiCad board)
At the start: 4 copper layers, 100 x 100 mm, 55 parts, among them J1 Serial port, J2 USB_B, J3 Expansion Header, SW1 RESET, SW2 RUN/STOP, SW3 SI, U1 74HC14, U2 IM6100, U3 2,4576 Mhz, U4 IM6101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

Commit message: HID board finalizing
Parts:
- removed HOLE1: MountingHole_3.2mm_M3, MountingHole:MountingHole_3.2mm_M3
- added JP6: onboard RAM enable, Connector_PinHeader_2.54mm:PinHeader_1x02_P2.54mm_Vertical, F.Cu at (171.4, 97.8)
- added R7: 10k, Resistor_THT:R_Axial_DIN0207_L6.3mm_D2.5mm_P7.62mm_Horizontal, F.Cu at (171.4, 129.5)
- added R8: 10k, Resistor_THT:R_Axial_DIN0207_L6.3mm_D2.5mm_P7.62mm_Horizontal, F.Cu at (106.7, 92.2)
- C10, C6, C7, C9: footprint Capacitor_THT:C_Disc_D3.0mm_W2.0mm_P2.50mm -> Capacitor_THT:C_Disc_D5.0mm_W2.5mm_P2.50mm
- C17: value 10nF -> 10nF 1000V
- J3: value Expansion Header -> Expansion port; footprint Connector_IDC:IDC-Header_2x15_P2.54mm_Vertical -> Connector_PinHeader_2.54mm:PinHeader_2x16_P2.54mm_Vertical
- U2: value IM6100 -> IM6101
- moved J3 3.54 mm to (104.1, 105.4)
- moved C8 2.82 mm to (171.4, 133.4)
- moved C12 2.52 mm to (171.4, 115.6)
- moved C13 2.52 mm to (171.4, 108.0)
- moved C2 2.52 mm to (171.4, 90.2)
Connections:
- J3 pad 10: DX10 -> /C0
- J3 pad 11: DX9 -> DX11
- J3 pad 12: DX8 -> DX10
- J3 pad 13: DX7 -> DX9
- J3 pad 14: DX6 -> DX8
- J3 pad 15: /DEVSEL -> DX7
- J3 pad 16: /SWSEL -> DX6
- J3 pad 17: XTA -> /DEVSEL
- J3 pad 18: LXMAR -> /SWSEL
- J3 pad 19: XTB -> XTA
- J3 pad 20: XTC -> LXMAR
- J3 pad 21: READ2 -> XTB
- J3 pad 22: WRITE2 -> XTC
- J3 pad 23: DX5 -> READ2
- J3 pad 24: DX4 -> WRITE2
- J3 pad 25: DX3 -> DX5
- J3 pad 26: DX2 -> DX4
- J3 pad 27: DX1 -> DX3
- J3 pad 28: DX0 -> DX2
- J3 pad 29: TXD -> DX1
- J3 pad 30: SENSE3/RXD -> DX0
- J3 pad 5: /SKP -> /WAIT
- J3 pad 6: /C2 -> /RESET
- J3 pad 7: /C1 -> /SKP
- J3 pad 8: /C0 -> /C2
- J3 pad 9: DX11 -> /C1
- U10 pad 15: Net-(U10-/S1) -> Net-(JP6-B)
- U2 pad 11: +5V -> /WAIT
- U7 pad 1: Net-(U10-/S1) -> Net-(JP6-A)
- U8 pad 15: Net-(U10-/S1) -> Net-(JP6-B)
- U9 pad 15: Net-(U10-/S1) -> Net-(JP6-B)
Routing:
- net Net-(JP6-B): track 0.00 -> 55.0 mm
- net /WAIT: track 0.00 -> 54.8 mm
- net Net-(U10-/S1): track 36.8 -> 0.00 mm
- net DX5: track 196.9 -> 232.9 mm, vias 3 -> 2
- net /RESET: track 42.6 -> 69.0 mm, vias 1 -> 0
- net XTC: track 167.6 -> 146.0 mm, vias 1 -> 0
- net DX8: track 244.2 -> 224.3 mm, vias 1 -> 0
- net DX4: track 185.5 -> 201.6 mm, vias 1 -> 0
- net LXMAR: track 173.7 -> 158.5 mm, vias 0 -> 1
- net DX7: track 234.2 -> 222.4 mm, vias 1 -> 0
- net DX11: track 225.5 -> 236.8 mm, vias 1 -> 0
- net DX3: track 145.2 -> 134.3 mm, vias 1 -> 2
- net /C0: track 46.3 -> 56.5 mm, vias 0 -> 1
- net DX2: track 117.9 -> 128.0 mm
- net /MEMSEL: track 145.5 -> 136.7 mm, vias 2 -> 0
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